File: left-display/left-display.kicad_pcb (KiCad board)
At the start: 2 copper layers, 80 x 20 mm, 49 parts, among them P1 CONN_6, P2 CONN_8

Commit message: Add comments for the fab regarding PCB properties.
Other:
- board text added: "Display PCB layer: * 1.55mm thickness * black soldermask * white silkscreen Insulator layer * 0.5mm thickness * etch away all copper from both sides * no soldermask * no silkscreen"
Changed lines of the file:
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@@
     (links 94)
     (no_connects 0)
-    (area 102.642669 89.033349 182.741571 109.132371)
+    (area 101.8176 46.0404 182.741571 109.132371)
     (thickness 1.6002)
-    (drawings 4)
+    (drawings 5)
     (tracks 356)
     (zones 0)
@@
       (usegerberextensions true)
       (excludeedgelayer true)
-      (linewidth 60)
+      (linewidth 0.150000)
       (plotframeref false)
       (viasonmask false)
@@
     )
   )
+  (gr_text "Display PCB layer:\n* 1.55mm thickness\n* black soldermask\n* white silkscreen\n\nInsulator layer\n* 0.5mm thickness\n* etch away all copper from both sides\n* no soldermask\n* no silkscreen" (at 102.59 63.12) (layer Cmts.User)
+    (effects (font (size 1.5 1.5) (thickness 0.3)) (justify left))
+  )
   (gr_line (start 102.6922 107.08386) (end 102.6922 109.08284) (angle 90) (layer Edge.Cuts) (width 0.09906))
