File: display-main/display-main.kicad_pcb (KiCad board)
At the start: 2 copper layers, 80 x 20 mm, 49 parts, among them P1 CONN_6, P2 CONN_8

Commit message: Update comments.
Other:
- board text added: "* 1.55mm board thickness * black soldermask * white silkscreen"
- board text removed: "Display PCB layer: * 1.55mm thickness * black soldermask * white silkscreen Insulator layer * 0.5mm thickness * etch away all copper from both sides * no soldermask * no silkscreen"
Changed lines of the file:
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@@
     (links 94)
     (no_connects 0)
-    (area 101.8176 46.0404 182.741571 109.132371)
+    (area 102.35 82.69 182.741571 109.132371)
     (thickness 1.6002)
     (drawings 5)
@@
   (page A4)
   (title_block
-    (title "Ultimate Hacking Keyboard - LED Display Board")
+    (title "Ultimate Hacking Keyboard - LED Display PCB Layer")
     (rev 3)
     (company "Ultimate Gadget Laboratories Kft.")
@@
     )
   )
-  (gr_text "Display PCB layer:\n* 1.55mm thickness\n* black soldermask\n* white silkscreen\n\nInsulator layer\n* 0.5mm thickness\n* etch away all copper from both sides\n* no soldermask\n* no silkscreen" (at 102.59 63.12) (layer Cmts.User)
+  (gr_text "* 1.55mm board thickness\n* black soldermask\n* white silkscreen\n" (at 102.5 84.19) (layer Cmts.User)
     (effects (font (size 1.5 1.5) (thickness 0.3)) (justify left))
   )
