File: right-connector/right-connector.kicad_pcb (KiCad board)
At the start: 2 copper layers, 18.7 x 3.2 mm, 0 parts

Commit message: Add comments for the fab regarding PCB properties.
Other:
- board text added: "* 1mm thickness * black soldermask * ENIG finish * no silkscreen"
Changed lines of the file:
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@@
     (links 0)
     (no_connects 0)
-    (area 138.386819 98.866959 157.099001 102.077521)
+    (area 138.0876 77.5104 160.889543 102.077521)
     (thickness 1.6002)
-    (drawings 5)
+    (drawings 6)
     (tracks 0)
     (zones 0)
@@
       (usegerberextensions true)
       (excludeedgelayer true)
-      (linewidth 60)
+      (linewidth 0.150000)
       (plotframeref false)
       (viasonmask false)
@@
     (add_net "")
   )
+  (gr_text "* 1mm thickness\n* black soldermask\n* ENIG finish\n* no silkscreen\n" (at 138.02 82.81) (layer Cmts.User)
+    (effects (font (size 1.5 1.5) (thickness 0.3)) (justify left))
+  )
   (gr_arc (start 156.09316 99.8728) (end 156.09316 98.87204) (angle 90) (layer Edge.Cuts) (width 0.01016))

Commit message: Update comments.
Other:
- board text added: "* 1mm board thickness * black soldermask * ENIG finish * no silkscreen"
- board text removed: "* 1mm thickness * black soldermask * ENIG finish * no silkscreen"
Changed lines of the file:
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@@
     (links 0)
     (no_connects 0)
-    (area 138.0876 77.5104 160.889543 102.077521)
+    (area 137.87 81.31 160.312857 102.077521)
     (thickness 1.6002)
     (drawings 6)
@@
     (add_net "")
   )
-  (gr_text "* 1mm thickness\n* black soldermask\n* ENIG finish\n* no silkscreen\n" (at 138.02 82.81) (layer Cmts.User)
+  (gr_text "* 1mm board thickness\n* black soldermask\n* ENIG finish\n* no silkscreen\n" (at 138.02 82.81) (layer Cmts.User)
     (effects (font (size 1.5 1.5) (thickness 0.3)) (justify left))
   )
