File: connectors/connectors.kicad_pcb (KiCad board)
At the start: 2 copper layers, 41.7 x 4.8 mm, 20 parts, among them P11 CONN_1, P12 CONN_1, P13 CONN_1, P14 CONN_1, P15 CONN_1, P21 CONN_1, P22 CONN_1, P23 CONN_1, P24 CONN_1, P25 CONN_1

Commit message: Update instructions on the comment layers.
Other:
- board text added: "design is 30mil-10mil-14mil trace-clearance-minimum_drill 2.5mm board thickness black solder mask ENIG finish no silk screen"
- board text removed: "* design is 30mil-10mil-14mil trace-clearance-minimum_drill * 2.5mm board thickness * black soldermask * ENIG finish * no silkscreen"
Changed lines of the file:
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@@
     (effects (font (size 2.032 1.524) (thickness 0.3048)) (justify mirror))
   )
-  (gr_text "* design is 30mil-10mil-14mil trace-clearance-minimum_drill\n* 2.5mm board thickness\n* black soldermask\n* ENIG finish\n* no silkscreen\n" (at 99.2124 87.7443) (layer Cmts.User)
+  (gr_text "design is 30mil-10mil-14mil trace-clearance-minimum_drill\n2.5mm board thickness\nblack solder mask\nENIG finish\nno silk screen" (at 99.2124 87.7443) (layer Cmts.User)
     (effects (font (size 1.5 1.5) (thickness 0.3)) (justify left))
   )
